File: kicad/COM.sch (KiCad schematic (older format))
At the start: 2 parts, among them P5 SWD, P6 UART

Commit message: add kicad .gitignore
Parts:
- P5: symbol CONN_01X05 -> KERISEv1-rescue:CONN_01X05
- P6: symbol CONN_01X04 -> KERISEv1-rescue:CONN_01X04
Changed lines of the file:
@@
-EESchema Schematic File Version 2
-LIBS:KERISEv1-rescue
-LIBS:74xgxx
-LIBS:74xx
-LIBS:ac-dc
-LIBS:actel
-LIBS:adc-dac
-LIBS:Altera
-LIBS:analog_devices
-LIBS:analog_switches
-LIBS:atmel
-LIBS:audio
-LIBS:brooktre
-LIBS:cmos_ieee
-LIBS:cmos4000
-LIBS:conn
-LIBS:contrib
-LIBS:cypress
-LIBS:dc-dc
-LIBS:device
-LIBS:digital-audio
-LIBS:diode
-LIBS:display
-LIBS:dsp
-LIBS:elec-unifil
-LIBS:ESD_Protection
-LIBS:ftdi
-LIBS:gennum
-LIBS:hc11
-LIBS:intel
-LIBS:interface
-LIBS:ir
-LIBS:Lattice
-LIBS:linear
-LIBS:maxim
-LIBS:memory
-LIBS:microchip
-LIBS:microchip_dspic33dsc
-LIBS:microchip_pic10mcu
-LIBS:microchip_pic12mcu
-LIBS:microchip_pic16mcu
-LIBS:microchip_pic18mcu
-LIBS:microchip_pic32mcu
-LIBS:microcontrollers
-LIBS:motor_drivers
-LIBS:motorola
-LIBS:msp430
-LIBS:nordicsemi
-LIBS:nxp_armmcu
-LIBS:onsemi
-LIBS:opto
-LIBS:Oscillators
-LIBS:philips
-LIBS:power
-LIBS:Power_Management
-LIBS:powerint
-LIBS:pspice
-LIBS:references
-LIBS:regul
-LIBS:relays
-LIBS:rfcom
-LIBS:sensors
-LIBS:silabs
-LIBS:siliconi
-LIBS:stm8
-LIBS:stm32
-LIBS:supertex
-LIBS:switches
-LIBS:texas
-LIBS:transf
-LIBS:transistors
-LIBS:ttl_ieee
-LIBS:valves
-LIBS:video
-LIBS:Xicor
-LIBS:xilinx
-LIBS:Zilog
-LIBS:KERISEv1
-LIBS:KERISEv1-cache
-EELAYER 25 0
+EESchema Schematic File Version 4
+EELAYER 30 0
 EELAYER END
 $Descr A4 11693 8268
@@
 SWO
 $Comp
-L GND #PWR98
+L power:GND #PWR98
 U 1 1 57CDA951
 P 4800 4500
@@
 	4900 4400 4700 4400
 $Comp
-L GND #PWR100
+L power:GND #PWR100
 U 1 1 57CDAC76
 P 5850 4500
@@
 	5850 4200 5750 4200
 $Comp
-L CONN_01X04 P6
+L KERISEv1-rescue:CONN_01X04 P6
 U 1 1 57CDB029
 P 5550 4250
@@
 	5950 4400 5750 4400
 $Comp
-L +5V #PWR99
+L power:+5V #PWR99
 U 1 1 57CDB089
 P 5850 4000
@@
 COM Port
 $Comp
-L CONN_01X05 P5
+L KERISEv1-rescue:CONN_01X05 P5
 U 1 1 57D2587E
 P 4500 4200
