File: kicad/IR_RCV.sch (KiCad schematic (older format))
At the start: 6 parts, among them U8 AD8604

Commit message: KiCadデータの名前をKERISEv1に変更
Changed lines of the file:
@@
 EESchema Schematic File Version 2
-LIBS:Mouse-01
 LIBS:74xgxx
 LIBS:74xx
@@
 LIBS:xilinx
 LIBS:Zilog
-LIBS:Mouse-01-cache
+LIBS:KERISEv1
+LIBS:kerikun11
+LIBS:KERISEv1-cache
 EELAYER 25 0
 EELAYER END
@@
 AR Path="/57CF292E/57CF0F37" Ref="D6"  Part="1"
 AR Path="/57CF2A30/57CF0F37" Ref="D7"  Part="1"
-F 0 "D7" H 4600 3950 50  0000 C CNN
+F 0 "D4" H 4600 3950 50  0000 C CNN
 F 1 "SFH213FA" H 4600 3750 50  0000 C CNN
 F 2 "kerikun11:Photo-5MM_Angle" H 4600 3850 50  0001 C CNN
@@
 $Comp
 L LM2902N U8
-U 4 1 57CF0F3E
+U 1 1 57CF0F3E
 P 5500 4000
 AR Path="/57CF0B09/57CF0F3E" Ref="U8"  Part="1"
@@
 F 2 "Housings_SSOP:TSSOP-14_4.4x5mm_Pitch0.65mm" H 5450 4100 50  0001 C CNN
 F 3 "" H 5550 4200 50  0000 C CNN
-	4    5500 4000
+	1    5500 4000
 	1    0    0    -1
 $EndComp
@@
 AR Path="/57CF292E/57CF0F45" Ref="C25"  Part="1"
 AR Path="/57CF2A30/57CF0F45" Ref="C27"  Part="1"
-F 0 "C27" H 4875 4200 50  0000 L CNN
+F 0 "C21" H 4875 4200 50  0000 L CNN
 F 1 "0.01u" H 4875 4000 50  0000 L CNN
 F 2 "Capacitors_SMD:C_0603" H 4888 3950 50  0001 C CNN
@@
 AR Path="/57CF292E/57CF0F4C" Ref="R13"  Part="1"
 AR Path="/57CF2A30/57CF0F4C" Ref="R15"  Part="1"
-F 0 "R15" V 4680 4650 50  0000 C CNN
+F 0 "R9" V 4680 4650 50  0000 C CNN
 F 1 "100k" V 4600 4650 50  0000 C CNN
 F 2 "Resistors_SMD:R_0603" V 4530 4650 50  0001 C CNN
@@
 AR Path="/57CF292E/57CF0F57" Ref="R12"  Part="1"
 AR Path="/57CF2A30/57CF0F57" Ref="R14"  Part="1"
-F 0 "R14" V 5730 3600 50  0000 C CNN
+F 0 "R8" V 5730 3600 50  0000 C CNN
 F 1 "220k" V 5650 3600 50  0000 C CNN
 F 2 "Resistors_SMD:R_0603" V 5580 3600 50  0001 C CNN
@@
 AR Path="/57CF292E/57CF0F5E" Ref="C24"  Part="1"
 AR Path="/57CF2A30/57CF0F5E" Ref="C26"  Part="1"
-F 0 "C26" H 5550 3500 50  0000 L CNN
+F 0 "C20" H 5550 3500 50  0000 L CNN
 F 1 "22p" H 5500 3300 50  0000 L CNN
 F 2 "Capacitors_SMD:C_0603" H 5688 3250 50  0001 C CNN
@@
 	4600 3200 4600 3700
 $Comp
-L +3.3VA #PWR059
+L +3.3VA #PWR55
 U 1 1 57CF0F71
 P 4600 3200
-AR Path="/57CF0B09/57CF0F71" Ref="#PWR059"  Part="1"
-AR Path="/57CF289D/57CF0F71" Ref="#PWR064"  Part="1"
-AR Path="/57CF292E/57CF0F71" Ref="#PWR069"  Part="1"
-AR Path="/57CF2A30/57CF0F71" Ref="#PWR074"  Part="1"
-F 0 "#PWR074" H 4750 3150 50  0001 C CNN
+AR Path="/57CF0B09/57CF0F71" Ref="#PWR55"  Part="1"
+AR Path="/57CF289D/57CF0F71" Ref="#PWR60"  Part="1"
+AR Path="/57CF292E/57CF0F71" Ref="#PWR65"  Part="1"
+AR Path="/57CF2A30/57CF0F71" Ref="#PWR70"  Part="1"
+F 0 "#PWR55" H 4750 3150 50  0001 C CNN
 F 1 "+3.3VA" H 4600 3300 50  0000 C CNN
 F 2 "" H 4600 3200 50  0000 C CNN
@@
 $EndComp
 $Comp
-L +3.3VA #PWR060
+L +3.3VA #PWR56
 U 1 1 57CF0F77
 P 5400 3200
-AR Path="/57CF0B09/57CF0F77" Ref="#PWR060"  Part="1"
-AR Path="/57CF289D/57CF0F77" Ref="#PWR065"  Part="1"
-AR Path="/57CF292E/57CF0F77" Ref="#PWR070"  Part="1"
-AR Path="/57CF2A30/57CF0F77" Ref="#PWR075"  Part="1"
-F 0 "#PWR075" H 5550 3150 50  0001 C CNN
+AR Path="/57CF0B09/57CF0F77" Ref="#PWR56"  Part="1"
+AR Path="/57CF289D/57CF0F77" Ref="#PWR61"  Part="1"
+AR Path="/57CF292E/57CF0F77" Ref="#PWR66"  Part="1"
+AR Path="/57CF2A30/57CF0F77" Ref="#PWR71"  Part="1"
+F 0 "#PWR56" H 5550 3150 50  0001 C CNN
 F 1 "+3.3VA" H 5400 3300 50  0000 C CNN
 F 2 "" H 5400 3200 50  0000 C CNN
@@
 $EndComp
 $Comp
-L +1.65VA #PWR061
+L +1.65VA #PWR57
 U 1 1 57CF0F7D
 P 4900 3800
-AR Path="/57CF0B09/57CF0F7D" Ref="#PWR061"  Part="1"
-AR Path="/57CF289D/57CF0F7D" Ref="#PWR066"  Part="1"
-AR Path="/57CF292E/57CF0F7D" Ref="#PWR071"  Part="1"
-AR Path="/57CF2A30/57CF0F7D" Ref="#PWR076"  Part="1"
-F 0 "#PWR076" H 5050 3750 50  0001 C CNN
+AR Path="/57CF0B09/57CF0F7D" Ref="#PWR57"  Part="1"
+AR Path="/57CF289D/57CF0F7D" Ref="#PWR62"  Part="1"
+AR Path="/57CF292E/57CF0F7D" Ref="#PWR67"  Part="1"
+AR Path="/57CF2A30/57CF0F7D" Ref="#PWR72"  Part="1"
+F 0 "#PWR57" H 5050 3750 50  0001 C CNN
 F 1 "+1.65VA" H 4900 3900 50  0000 C CNN
 F 2 "" H 4900 3800 50  0000 C CNN
@@
 	4900 3900 5200 3900
 $Comp
-L GND #PWR062
+L GND #PWR58
 U 1 1 57CF0F85
 P 4600 4900
-AR Path="/57CF0B09/57CF0F85" Ref="#PWR062"  Part="1"
-AR Path="/57CF289D/57CF0F85" Ref="#PWR067"  Part="1"
-AR Path="/57CF292E/57CF0F85" Ref="#PWR072"  Part="1"
-AR Path="/57CF2A30/57CF0F85" Ref="#PWR077"  Part="1"
-F 0 "#PWR077" H 4600 4650 50  0001 C CNN
+AR Path="/57CF0B09/57CF0F85" Ref="#PWR58"  Part="1"
+AR Path="/57CF289D/57CF0F85" Ref="#PWR63"  Part="1"
+AR Path="/57CF292E/57CF0F85" Ref="#PWR68"  Part="1"
+AR Path="/57CF2A30/57CF0F85" Ref="#PWR73"  Part="1"
+F 0 "#PWR58" H 4600 4650 50  0001 C CNN
 F 1 "GND" H 4600 4750 50  0000 C CNN
 F 2 "" H 4600 4900 50  0000 C CNN
@@
 	4600 4900 4600 4800
 $Comp
-L GND #PWR063
+L GND #PWR59
 U 1 1 57CF0F8C
 P 5400 4900
-AR Path="/57CF0B09/57CF0F8C" Ref="#PWR063"  Part="1"
-AR Path="/57CF289D/57CF0F8C" Ref="#PWR068"  Part="1"
-AR Path="/57CF292E/57CF0F8C" Ref="#PWR073"  Part="1"
-AR Path="/57CF2A30/57CF0F8C" Ref="#PWR078"  Part="1"
-F 0 "#PWR078" H 5400 4650 50  0001 C CNN
+AR Path="/57CF0B09/57CF0F8C" Ref="#PWR59"  Part="1"
+AR Path="/57CF289D/57CF0F8C" Ref="#PWR64"  Part="1"
+AR Path="/57CF292E/57CF0F8C" Ref="#PWR69"  Part="1"
+AR Path="/57CF2A30/57CF0F8C" Ref="#PWR74"  Part="1"
+F 0 "#PWR59" H 5400 4650 50  0001 C CNN
 F 1 "GND" H 5400 4750 50  0000 C CNN
 F 2 "" H 5400 4900 50  0000 C CNN
@@
 Text HLabel 6000 4000 2    60   Input ~ 0
 IR_RCV
-Text Notes 3700 2800 0    100  ~ 0
+Text Notes 4000 2900 0    100  ~ 0
 IR Receiver
 $EndSCHEMATC

Commit message: 回路図を修正
電源スイッチにPchFETを挿入
赤外線LED用FETのゲートをプルダウン
Parts:
- renumbered C20 to C22, R9 to R10, R8 to R11
Other:
- note added: "IR Receiver\nKERI's Lab\n2016.12.28"
- note removed: "IR Receiver"
Changed lines of the file:
@@
 EESchema Schematic File Version 2
+LIBS:KERISEv1-rescue
 LIBS:74xgxx
 LIBS:74xx
@@
 LIBS:cmos4000
 LIBS:conn
-LIBS:connectors
 LIBS:contrib
 LIBS:cypress
@@
 LIBS:ftdi
 LIBS:gennum
-LIBS:graphic
 LIBS:hc11
-LIBS:ic-cpu
-LIBS:ic-io
-LIBS:ic-misc
-LIBS:ic-power
 LIBS:intel
 LIBS:interface
@@
 LIBS:Lattice
 LIBS:linear
-LIBS:logo
 LIBS:maxim
 LIBS:memory
@@
 LIBS:opto
 LIBS:Oscillators
-LIBS:passive
 LIBS:philips
 LIBS:power
@@
 LIBS:Zilog
 LIBS:KERISEv1
-LIBS:kerikun11
 LIBS:KERISEv1-cache
 EELAYER 25 0
@@
 $EndComp
 $Comp
-L R R9
+L R R10
 U 1 1 57CF0F4C
 P 4600 4650
-AR Path="/57CF0B09/57CF0F4C" Ref="R9"  Part="1"
-AR Path="/57CF289D/57CF0F4C" Ref="R11"  Part="1"
-AR Path="/57CF292E/57CF0F4C" Ref="R13"  Part="1"
-AR Path="/57CF2A30/57CF0F4C" Ref="R15"  Part="1"
-F 0 "R9" V 4680 4650 50  0000 C CNN
+AR Path="/57CF0B09/57CF0F4C" Ref="R10"  Part="1"
+AR Path="/57CF289D/57CF0F4C" Ref="R12"  Part="1"
+AR Path="/57CF292E/57CF0F4C" Ref="R14"  Part="1"
+AR Path="/57CF2A30/57CF0F4C" Ref="R16"  Part="1"
+F 0 "R10" V 4680 4650 50  0000 C CNN
 F 1 "100k" V 4600 4650 50  0000 C CNN
 F 2 "Resistors_SMD:R_0603" V 4530 4650 50  0001 C CNN
@@
 Connection ~ 4600 4100
 $Comp
-L R R8
+L R R11
 U 1 1 57CF0F57
 P 5650 3600
-AR Path="/57CF0B09/57CF0F57" Ref="R8"  Part="1"
-AR Path="/57CF289D/57CF0F57" Ref="R10"  Part="1"
-AR Path="/57CF292E/57CF0F57" Ref="R12"  Part="1"
-AR Path="/57CF2A30/57CF0F57" Ref="R14"  Part="1"
-F 0 "R8" V 5730 3600 50  0000 C CNN
+AR Path="/57CF0B09/57CF0F57" Ref="R11"  Part="1"
+AR Path="/57CF289D/57CF0F57" Ref="R13"  Part="1"
+AR Path="/57CF292E/57CF0F57" Ref="R15"  Part="1"
+AR Path="/57CF2A30/57CF0F57" Ref="R17"  Part="1"
+F 0 "R11" V 5730 3600 50  0000 C CNN
 F 1 "220k" V 5650 3600 50  0000 C CNN
 F 2 "Resistors_SMD:R_0603" V 5580 3600 50  0001 C CNN
@@
 $EndComp
 $Comp
-L C C20
+L C C22
 U 1 1 57CF0F5E
 P 5650 3400
-AR Path="/57CF0B09/57CF0F5E" Ref="C20"  Part="1"
-AR Path="/57CF289D/57CF0F5E" Ref="C22"  Part="1"
-AR Path="/57CF292E/57CF0F5E" Ref="C24"  Part="1"
-AR Path="/57CF2A30/57CF0F5E" Ref="C26"  Part="1"
-F 0 "C20" H 5550 3500 50  0000 L CNN
+AR Path="/57CF0B09/57CF0F5E" Ref="C22"  Part="1"
+AR Path="/57CF289D/57CF0F5E" Ref="C24"  Part="1"
+AR Path="/57CF292E/57CF0F5E" Ref="C26"  Part="1"
+AR Path="/57CF2A30/57CF0F5E" Ref="C28"  Part="1"
+F 0 "C22" H 5550 3500 50  0000 L CNN
 F 1 "22p" H 5500 3300 50  0000 L CNN
 F 2 "Capacitors_SMD:C_0603" H 5688 3250 50  0001 C CNN
@@
 	4600 3200 4600 3700
 $Comp
-L +3.3VA #PWR55
+L +3.3VA-RESCUE-KERISEv1 #PWR58
 U 1 1 57CF0F71
 P 4600 3200
-AR Path="/57CF0B09/57CF0F71" Ref="#PWR55"  Part="1"
-AR Path="/57CF289D/57CF0F71" Ref="#PWR60"  Part="1"
-AR Path="/57CF292E/57CF0F71" Ref="#PWR65"  Part="1"
-AR Path="/57CF2A30/57CF0F71" Ref="#PWR70"  Part="1"
-F 0 "#PWR55" H 4750 3150 50  0001 C CNN
+AR Path="/57CF0B09/57CF0F71" Ref="#PWR58"  Part="1"
+AR Path="/57CF289D/57CF0F71" Ref="#PWR63"  Part="1"
+AR Path="/57CF292E/57CF0F71" Ref="#PWR68"  Part="1"
+AR Path="/57CF2A30/57CF0F71" Ref="#PWR73"  Part="1"
+F 0 "#PWR58" H 4750 3150 50  0001 C CNN
 F 1 "+3.3VA" H 4600 3300 50  0000 C CNN
 F 2 "" H 4600 3200 50  0000 C CNN
@@
 $EndComp
 $Comp
-L +3.3VA #PWR56
+L +3.3VA-RESCUE-KERISEv1 #PWR61
 U 1 1 57CF0F77
 P 5400 3200
-AR Path="/57CF0B09/57CF0F77" Ref="#PWR56"  Part="1"
-AR Path="/57CF289D/57CF0F77" Ref="#PWR61"  Part="1"
-AR Path="/57CF292E/57CF0F77" Ref="#PWR66"  Part="1"
-AR Path="/57CF2A30/57CF0F77" Ref="#PWR71"  Part="1"
-F 0 "#PWR56" H 5550 3150 50  0001 C CNN
+AR Path="/57CF0B09/57CF0F77" Ref="#PWR61"  Part="1"
+AR Path="/57CF289D/57CF0F77" Ref="#PWR66"  Part="1"
+AR Path="/57CF292E/57CF0F77" Ref="#PWR71"  Part="1"
+AR Path="/57CF2A30/57CF0F77" Ref="#PWR76"  Part="1"
+F 0 "#PWR61" H 5550 3150 50  0001 C CNN
 F 1 "+3.3VA" H 5400 3300 50  0000 C CNN
 F 2 "" H 5400 3200 50  0000 C CNN
@@
 $EndComp
 $Comp
-L +1.65VA #PWR57
+L +1.65VA #PWR60
 U 1 1 57CF0F7D
 P 4900 3800
-AR Path="/57CF0B09/57CF0F7D" Ref="#PWR57"  Part="1"
-AR Path="/57CF289D/57CF0F7D" Ref="#PWR62"  Part="1"
-AR Path="/57CF292E/57CF0F7D" Ref="#PWR67"  Part="1"
-AR Path="/57CF2A30/57CF0F7D" Ref="#PWR72"  Part="1"
-F 0 "#PWR57" H 5050 3750 50  0001 C CNN
+AR Path="/57CF0B09/57CF0F7D" Ref="#PWR60"  Part="1"
+AR Path="/57CF289D/57CF0F7D" Ref="#PWR65"  Part="1"
+AR Path="/57CF292E/57CF0F7D" Ref="#PWR70"  Part="1"
+AR Path="/57CF2A30/57CF0F7D" Ref="#PWR75"  Part="1"
+F 0 "#PWR60" H 5050 3750 50  0001 C CNN
 F 1 "+1.65VA" H 4900 3900 50  0000 C CNN
 F 2 "" H 4900 3800 50  0000 C CNN
@@
 	4900 3900 5200 3900
 $Comp
-L GND #PWR58
+L GND #PWR59
 U 1 1 57CF0F85
 P 4600 4900
-AR Path="/57CF0B09/57CF0F85" Ref="#PWR58"  Part="1"
-AR Path="/57CF289D/57CF0F85" Ref="#PWR63"  Part="1"
-AR Path="/57CF292E/57CF0F85" Ref="#PWR68"  Part="1"
-AR Path="/57CF2A30/57CF0F85" Ref="#PWR73"  Part="1"
-F 0 "#PWR58" H 4600 4650 50  0001 C CNN
+AR Path="/57CF0B09/57CF0F85" Ref="#PWR59"  Part="1"
+AR Path="/57CF289D/57CF0F85" Ref="#PWR64"  Part="1"
+AR Path="/57CF292E/57CF0F85" Ref="#PWR69"  Part="1"
+AR Path="/57CF2A30/57CF0F85" Ref="#PWR74"  Part="1"
+F 0 "#PWR59" H 4600 4650 50  0001 C CNN
 F 1 "GND" H 4600 4750 50  0000 C CNN
 F 2 "" H 4600 4900 50  0000 C CNN
@@
 	4600 4900 4600 4800
 $Comp
-L GND #PWR59
+L GND #PWR62
 U 1 1 57CF0F8C
 P 5400 4900
-AR Path="/57CF0B09/57CF0F8C" Ref="#PWR59"  Part="1"
-AR Path="/57CF289D/57CF0F8C" Ref="#PWR64"  Part="1"
-AR Path="/57CF292E/57CF0F8C" Ref="#PWR69"  Part="1"
-AR Path="/57CF2A30/57CF0F8C" Ref="#PWR74"  Part="1"
-F 0 "#PWR59" H 5400 4650 50  0001 C CNN
+AR Path="/57CF0B09/57CF0F8C" Ref="#PWR62"  Part="1"
+AR Path="/57CF289D/57CF0F8C" Ref="#PWR67"  Part="1"
+AR Path="/57CF292E/57CF0F8C" Ref="#PWR72"  Part="1"
+AR Path="/57CF2A30/57CF0F8C" Ref="#PWR77"  Part="1"
+F 0 "#PWR62" H 5400 4650 50  0001 C CNN
 F 1 "GND" H 5400 4750 50  0000 C CNN
 F 2 "" H 5400 4900 50  0000 C CNN
@@
 Text HLabel 6000 4000 2    60   Input ~ 0
 IR_RCV
-Text Notes 4000 2900 0    100  ~ 0
-IR Receiver
+Text Notes 3500 3350 0    100  ~ 0
+IR Receiver\nKERI's Lab\n2016.12.28
 $EndSCHEMATC

Commit message: add kicad .gitignore
Parts:
- C21, C22: symbol C -> KERISEv1-rescue:C
- D4: symbol D -> KERISEv1-rescue:D
- R10, R11: symbol R -> KERISEv1-rescue:R
- U8: symbol LM2902N -> KERISEv1-rescue:LM2902N
Changed lines of the file:
@@
-EESchema Schematic File Version 2
-LIBS:KERISEv1-rescue
-LIBS:74xgxx
-LIBS:74xx
-LIBS:ac-dc
-LIBS:actel
-LIBS:adc-dac
-LIBS:Altera
-LIBS:analog_devices
-LIBS:analog_switches
-LIBS:atmel
-LIBS:audio
-LIBS:brooktre
-LIBS:cmos_ieee
-LIBS:cmos4000
-LIBS:conn
-LIBS:contrib
-LIBS:cypress
-LIBS:dc-dc
-LIBS:device
-LIBS:digital-audio
-LIBS:diode
-LIBS:display
-LIBS:dsp
-LIBS:elec-unifil
-LIBS:ESD_Protection
-LIBS:ftdi
-LIBS:gennum
-LIBS:hc11
-LIBS:intel
-LIBS:interface
-LIBS:ir
-LIBS:Lattice
-LIBS:linear
-LIBS:maxim
-LIBS:memory
-LIBS:microchip
-LIBS:microchip_dspic33dsc
-LIBS:microchip_pic10mcu
-LIBS:microchip_pic12mcu
-LIBS:microchip_pic16mcu
-LIBS:microchip_pic18mcu
-LIBS:microchip_pic32mcu
-LIBS:microcontrollers
-LIBS:motor_drivers
-LIBS:motorola
-LIBS:msp430
-LIBS:nordicsemi
-LIBS:nxp_armmcu
-LIBS:onsemi
-LIBS:opto
-LIBS:Oscillators
-LIBS:philips
-LIBS:power
-LIBS:Power_Management
-LIBS:powerint
-LIBS:pspice
-LIBS:references
-LIBS:regul
-LIBS:relays
-LIBS:rfcom
-LIBS:sensors
-LIBS:silabs
-LIBS:siliconi
-LIBS:stm8
-LIBS:stm32
-LIBS:supertex
-LIBS:switches
-LIBS:texas
-LIBS:transf
-LIBS:transistors
-LIBS:ttl_ieee
-LIBS:valves
-LIBS:video
-LIBS:Xicor
-LIBS:xilinx
-LIBS:Zilog
-LIBS:KERISEv1
-LIBS:KERISEv1-cache
-EELAYER 25 0
+EESchema Schematic File Version 4
+EELAYER 30 0
 EELAYER END
 $Descr A4 11693 8268
@@
 $EndDescr
 $Comp
-L D D4
+L KERISEv1-rescue:D D4
 U 1 1 57CF0F37
 P 4600 3850
@@
 AR Path="/57CF292E/57CF0F37" Ref="D6"  Part="1"
 AR Path="/57CF2A30/57CF0F37" Ref="D7"  Part="1"
+AR Path="/57CF0F37" Ref="D4"  Part="1"
 F 0 "D4" H 4600 3950 50  0000 C CNN
 F 1 "SFH213FA" H 4600 3750 50  0000 C CNN
@@
 $EndComp
 $Comp
-L LM2902N U8
+L KERISEv1-rescue:LM2902N U8
 U 1 1 57CF0F3E
 P 5500 4000
@@
 AR Path="/57CF292E/57CF0F3E" Ref="U8"  Part="3"
 AR Path="/57CF2A30/57CF0F3E" Ref="U8"  Part="4"
+AR Path="/57CF0F3E" Ref="U8"  Part="1"
 F 0 "U8" H 5550 4200 50  0000 C CNN
 F 1 "AD8604" H 5650 3800 50  0000 C CNN
@@
 $EndComp
 $Comp
-L C C21
+L KERISEv1-rescue:C C21
 U 1 1 57CF0F45
 P 4850 4100
@@
 AR Path="/57CF292E/57CF0F45" Ref="C25"  Part="1"
 AR Path="/57CF2A30/57CF0F45" Ref="C27"  Part="1"
+AR Path="/57CF0F45" Ref="C21"  Part="1"
 F 0 "C21" H 4875 4200 50  0000 L CNN
 F 1 "0.01u" H 4875 4000 50  0000 L CNN
@@
 $EndComp
 $Comp
-L R R10
+L KERISEv1-rescue:R R10
 U 1 1 57CF0F4C
 P 4600 4650
@@
 AR Path="/57CF292E/57CF0F4C" Ref="R14"  Part="1"
 AR Path="/57CF2A30/57CF0F4C" Ref="R16"  Part="1"
+AR Path="/57CF0F4C" Ref="R10"  Part="1"
 F 0 "R10" V 4680 4650 50  0000 C CNN
 F 1 "100k" V 4600 4650 50  0000 C CNN
@@
 Connection ~ 4600 4100
 $Comp
-L R R11
+L KERISEv1-rescue:R R11
 U 1 1 57CF0F57
 P 5650 3600
@@
 AR Path="/57CF292E/57CF0F57" Ref="R15"  Part="1"
 AR Path="/57CF2A30/57CF0F57" Ref="R17"  Part="1"
+AR Path="/57CF0F57" Ref="R11"  Part="1"
 F 0 "R11" V 5730 3600 50  0000 C CNN
 F 1 "220k" V 5650 3600 50  0000 C CNN
@@
 $EndComp
 $Comp
-L C C22
+L KERISEv1-rescue:C C22
 U 1 1 57CF0F5E
 P 5650 3400
@@
 AR Path="/57CF292E/57CF0F5E" Ref="C26"  Part="1"
 AR Path="/57CF2A30/57CF0F5E" Ref="C28"  Part="1"
+AR Path="/57CF0F5E" Ref="C22"  Part="1"
 F 0 "C22" H 5550 3500 50  0000 L CNN
 F 1 "22p" H 5500 3300 50  0000 L CNN
@@
 	4600 3200 4600 3700
 $Comp
-L +3.3VA-RESCUE-KERISEv1 #PWR58
+L KERISEv1-rescue:+3.3VA-RESCUE-KERISEv1 #PWR58
 U 1 1 57CF0F71
 P 4600 3200
@@
 $EndComp
 $Comp
-L +3.3VA-RESCUE-KERISEv1 #PWR61
+L KERISEv1-rescue:+3.3VA-RESCUE-KERISEv1 #PWR61
 U 1 1 57CF0F77
 P 5400 3200
@@
 $EndComp
 $Comp
-L +1.65VA #PWR60
+L KERISEv1:+1.65VA #PWR60
 U 1 1 57CF0F7D
 P 4900 3800
@@
 	4900 3900 5200 3900
 $Comp
-L GND #PWR59
+L power:GND #PWR59
 U 1 1 57CF0F85
 P 4600 4900
@@
 	4600 4900 4600 4800
 $Comp
-L GND #PWR62
+L power:GND #PWR62
 U 1 1 57CF0F8C
 P 5400 4900
