File: kicad/KERISEv1.sch (KiCad schematic (older format))
At the start: 11 parts, among them SW1 RESET, U1 STM32F405RGTx

Commit message: KiCadデータの名前をKERISEv1に変更
Parts:
- U1: footprint Housings_QFP:LQFP-64_10x10mm_Pitch0.5mm -> LQFP64
Changed lines of the file:
@@
 EESchema Schematic File Version 2
-LIBS:Mouse-01
 LIBS:74xgxx
 LIBS:74xx
@@
 LIBS:xilinx
 LIBS:Zilog
-LIBS:Mouse-01-cache
+LIBS:KERISEv1
+LIBS:kerikun11
+LIBS:KERISEv1-cache
 EELAYER 25 0
 EELAYER END
@@
 $EndDescr
 $Comp
-L STM32F405RGTx U1
-U 1 1 57C8ED63
-P 7600 3600
-F 0 "U1" H 5050 6550 50  0000 L BNN
-F 1 "STM32F405RGTx" H 5650 6400 50  0000 R BNN
-F 2 "Housings_QFP:LQFP-64_10x10mm_Pitch0.5mm" H 6850 1050 50  0000 R TNN
-F 3 "" H 6050 4800 50  0000 C CNN
-	1    7600 3600
-	1    0    0    -1
-$EndComp
-$Comp
-L +3.3V #PWR01
+L +3.3V #PWR1
 U 1 1 57C90296
 P 4800 1000
-F 0 "#PWR01" H 4800 850 50  0001 C CNN
+F 0 "#PWR1" H 4800 850 50  0001 C CNN
 F 1 "+3.3V" H 4800 1140 50  0000 C CNN
 F 2 "" H 4800 1000 50  0000 C CNN
@@
 $EndComp
 $Comp
-L GND #PWR02
+L GND #PWR4
 U 1 1 57C96070
 P 4600 3700
-F 0 "#PWR02" H 4600 3450 50  0001 C CNN
+F 0 "#PWR4" H 4600 3450 50  0001 C CNN
 F 1 "GND" H 4600 3550 50  0000 C CNN
 F 2 "" H 4600 3700 50  0000 C CNN
@@
 $EndComp
 $Comp
-L GND #PWR03
+L GND #PWR3
 U 1 1 57C960BE
 P 4300 3700
-F 0 "#PWR03" H 4300 3450 50  0001 C CNN
+F 0 "#PWR3" H 4300 3450 50  0001 C CNN
 F 1 "GND" H 4300 3550 50  0000 C CNN
 F 2 "" H 4300 3700 50  0000 C CNN
@@
 $EndComp
 $Comp
-L GND #PWR04
+L GND #PWR6
 U 1 1 57C99E1F
 P 4300 5100
-F 0 "#PWR04" H 4300 4850 50  0001 C CNN
+F 0 "#PWR6" H 4300 4850 50  0001 C CNN
 F 1 "GND" H 4300 4950 50  0000 C CNN
 F 2 "" H 4300 5100 50  0000 C CNN
@@
 $EndComp
 $Comp
-L GND #PWR05
+L GND #PWR7
 U 1 1 57C9A3C2
 P 4800 6100
-F 0 "#PWR05" H 4800 5850 50  0001 C CNN
+F 0 "#PWR7" H 4800 5850 50  0001 C CNN
 F 1 "GND" H 4800 5950 50  0000 C CNN
 F 2 "" H 4800 6100 50  0000 C CNN
@@
 $EndComp
 $Comp
-L GND #PWR06
+L GND #PWR5
 U 1 1 57CA25EF
 P 4800 3900
-F 0 "#PWR06" H 4800 3650 50  0001 C CNN
+F 0 "#PWR5" H 4800 3650 50  0001 C CNN
 F 1 "GND" H 4800 3750 50  0000 C CNN
 F 2 "" H 4800 3900 50  0000 C CNN
@@
 $EndComp
 $Comp
-L GND #PWR07
+L GND #PWR2
 U 1 1 57CDA895
 P 4300 2600
-F 0 "#PWR07" H 4300 2350 50  0001 C CNN
+F 0 "#PWR2" H 4300 2350 50  0001 C CNN
 F 1 "GND" H 4300 2450 50  0000 C CNN
 F 2 "" H 4300 2600 50  0000 C CNN
@@
 SPEAKER
 $Comp
-L PWR_FLAG #FLG08
+L PWR_FLAG #FLG1
 U 1 1 57D09A39
 P 4700 4450
-F 0 "#FLG08" H 4700 4545 50  0001 C CNN
+F 0 "#FLG1" H 4700 4545 50  0001 C CNN
 F 1 "PWR_FLAG" H 4700 4630 50  0000 C CNN
 F 2 "" H 4700 4450 50  0000 C CNN
@@
 $EndComp
 $Comp
-L PWR_FLAG #FLG09
+L PWR_FLAG #FLG2
 U 1 1 57D180C1
 P 4700 4900
-F 0 "#FLG09" H 4700 4995 50  0001 C CNN
+F 0 "#FLG2" H 4700 4995 50  0001 C CNN
 F 1 "PWR_FLAG" H 4700 5080 50  0000 C CNN
 F 2 "" H 4700 4900 50  0000 C CNN
@@
 Text Notes 700  800  0    100  ~ 0
 Main
+$Comp
+L STM32F405RGTx U1
+U 1 1 5862791B
+P 7600 3600
+F 0 "U1" H 5050 6550 50  0000 L BNN
+F 1 "STM32F405RGTx" H 5650 6400 50  0000 R BNN
+F 2 "LQFP64" H 5650 6350 50  0000 R TNN
+F 3 "" H 6050 4800 50  0000 C CNN
+	1    7600 3600
+	1    0    0    -1
+$EndComp
 $EndSCHEMATC

Commit message: 回路図を修正
電源スイッチにPchFETを挿入
赤外線LED用FETのゲートをプルダウン
Parts:
- U1: symbol STM32F405RGTx -> STM32F405RGTx-RESCUE-KERISEv1
- renumbered C8 to C7, C9 to C8, C7 to C9
Changed lines of the file:
@@
 EESchema Schematic File Version 2
+LIBS:KERISEv1-rescue
 LIBS:74xgxx
 LIBS:74xx
@@
 LIBS:cmos4000
 LIBS:conn
-LIBS:connectors
 LIBS:contrib
 LIBS:cypress
@@
 LIBS:ftdi
 LIBS:gennum
-LIBS:graphic
 LIBS:hc11
-LIBS:ic-cpu
-LIBS:ic-io
-LIBS:ic-misc
-LIBS:ic-power
 LIBS:intel
 LIBS:interface
@@
 LIBS:Lattice
 LIBS:linear
-LIBS:logo
 LIBS:maxim
 LIBS:memory
@@
 LIBS:opto
 LIBS:Oscillators
-LIBS:passive
 LIBS:philips
 LIBS:power
@@
 LIBS:Zilog
 LIBS:KERISEv1
-LIBS:kerikun11
 LIBS:KERISEv1-cache
 EELAYER 25 0
@@
 $EndDescr
 $Comp
-L +3.3V #PWR1
+L +3.3V #PWR5
 U 1 1 57C90296
 P 4800 1000
-F 0 "#PWR1" H 4800 850 50  0001 C CNN
+F 0 "#PWR5" H 4800 850 50  0001 C CNN
 F 1 "+3.3V" H 4800 1140 50  0000 C CNN
 F 2 "" H 4800 1000 50  0000 C CNN
@@
 $EndComp
 $Comp
-L C_Small C9
+L C_Small C8
 U 1 1 57C91C59
 P 4500 4800
-F 0 "C9" H 4510 4870 50  0000 L CNN
+F 0 "C8" H 4510 4870 50  0000 L CNN
 F 1 "2.2u" H 4510 4720 50  0000 L CNN
 F 2 "Capacitors_SMD:C_0603" H 4500 4800 50  0001 C CNN
@@
 $EndComp
 $Comp
-L C_Small C8
+L C_Small C7
 U 1 1 57C928EA
 P 4500 4550
-F 0 "C8" H 4510 4620 50  0000 L CNN
+F 0 "C7" H 4510 4620 50  0000 L CNN
 F 1 "2.2u" H 4510 4470 50  0000 L CNN
 F 2 "Capacitors_SMD:C_0603" H 4500 4550 50  0001 C CNN
@@
 $EndComp
 $Comp
-L GND #PWR3
+L GND #PWR2
 U 1 1 57C960BE
 P 4300 3700
-F 0 "#PWR3" H 4300 3450 50  0001 C CNN
+F 0 "#PWR2" H 4300 3450 50  0001 C CNN
 F 1 "GND" H 4300 3550 50  0000 C CNN
 F 2 "" H 4300 3700 50  0000 C CNN
@@
 $EndComp
 $Comp
-L GND #PWR6
+L GND #PWR3
 U 1 1 57C99E1F
 P 4300 5100
-F 0 "#PWR6" H 4300 4850 50  0001 C CNN
+F 0 "#PWR3" H 4300 4850 50  0001 C CNN
 F 1 "GND" H 4300 4950 50  0000 C CNN
 F 2 "" H 4300 5100 50  0000 C CNN
@@
 $EndComp
 $Comp
-L GND #PWR5
+L GND #PWR6
 U 1 1 57CA25EF
 P 4800 3900
-F 0 "#PWR5" H 4800 3650 50  0001 C CNN
+F 0 "#PWR6" H 4800 3650 50  0001 C CNN
 F 1 "GND" H 4800 3750 50  0000 C CNN
 F 2 "" H 4800 3900 50  0000 C CNN
@@
 $EndComp
 $Comp
-L GND #PWR2
+L GND #PWR1
 U 1 1 57CDA895
 P 4300 2600
-F 0 "#PWR2" H 4300 2350 50  0001 C CNN
+F 0 "#PWR1" H 4300 2350 50  0001 C CNN
 F 1 "GND" H 4300 2450 50  0000 C CNN
 F 2 "" H 4300 2600 50  0000 C CNN
@@
 RESET
 $Comp
-L C C7
+L C C9
 U 1 1 57CDEB3C
 P 4600 3300
-F 0 "C7" H 4625 3400 50  0000 L CNN
+F 0 "C9" H 4625 3400 50  0000 L CNN
 F 1 "0.1u" H 4625 3200 50  0000 L CNN
 F 2 "Capacitors_SMD:C_0603" H 4638 3150 50  0001 C CNN
@@
 Main
 $Comp
-L STM32F405RGTx U1
+L STM32F405RGTx-RESCUE-KERISEv1 U1
 U 1 1 5862791B
 P 7600 3600

Commit message: add kicad .gitignore
Parts:
- C1, C2, C3, C4, C5, C6, C7, C8: symbol C_Small -> KERISEv1-rescue:C_Small
- C9: symbol C -> KERISEv1-rescue:C
- SW1: symbol Tactile_SW_4P -> KERISEv1:Tactile_SW_4P
- U1: symbol STM32F405RGTx-RESCUE-KERISEv1 -> KERISEv1-rescue:STM32F405RGTx-RESCUE-KERISEv1
Changed lines of the file:
@@
-EESchema Schematic File Version 2
-LIBS:KERISEv1-rescue
-LIBS:74xgxx
-LIBS:74xx
-LIBS:ac-dc
-LIBS:actel
-LIBS:adc-dac
-LIBS:Altera
-LIBS:analog_devices
-LIBS:analog_switches
-LIBS:atmel
-LIBS:audio
-LIBS:brooktre
-LIBS:cmos_ieee
-LIBS:cmos4000
-LIBS:conn
-LIBS:contrib
-LIBS:cypress
-LIBS:dc-dc
-LIBS:device
-LIBS:digital-audio
-LIBS:diode
-LIBS:display
-LIBS:dsp
-LIBS:elec-unifil
-LIBS:ESD_Protection
-LIBS:ftdi
-LIBS:gennum
-LIBS:hc11
-LIBS:intel
-LIBS:interface
-LIBS:ir
-LIBS:Lattice
-LIBS:linear
-LIBS:maxim
-LIBS:memory
-LIBS:microchip
-LIBS:microchip_dspic33dsc
-LIBS:microchip_pic10mcu
-LIBS:microchip_pic12mcu
-LIBS:microchip_pic16mcu
-LIBS:microchip_pic18mcu
-LIBS:microchip_pic32mcu
-LIBS:microcontrollers
-LIBS:motor_drivers
-LIBS:motorola
-LIBS:msp430
-LIBS:nordicsemi
-LIBS:nxp_armmcu
-LIBS:onsemi
-LIBS:opto
-LIBS:Oscillators
-LIBS:philips
-LIBS:power
-LIBS:Power_Management
-LIBS:powerint
-LIBS:pspice
-LIBS:references
-LIBS:regul
-LIBS:relays
-LIBS:rfcom
-LIBS:sensors
-LIBS:silabs
-LIBS:siliconi
-LIBS:stm8
-LIBS:stm32
-LIBS:supertex
-LIBS:switches
-LIBS:texas
-LIBS:transf
-LIBS:transistors
-LIBS:ttl_ieee
-LIBS:valves
-LIBS:video
-LIBS:Xicor
-LIBS:xilinx
-LIBS:Zilog
-LIBS:KERISEv1
-LIBS:KERISEv1-cache
-EELAYER 25 0
+EESchema Schematic File Version 4
+EELAYER 30 0
 EELAYER END
 $Descr A4 11693 8268
@@
 $EndDescr
 $Comp
-L +3.3V #PWR5
+L power:+3.3V #PWR5
 U 1 1 57C90296
 P 4800 1000
@@
 $EndComp
 $Comp
-L C_Small C8
+L KERISEv1-rescue:C_Small C8
 U 1 1 57C91C59
 P 4500 4800
@@
 $EndComp
 $Comp
-L C_Small C7
+L KERISEv1-rescue:C_Small C7
 U 1 1 57C928EA
 P 4500 4550
@@
 $EndComp
 $Comp
-L GND #PWR4
+L power:GND #PWR4
 U 1 1 57C96070
 P 4600 3700
@@
 $EndComp
 $Comp
-L GND #PWR2
+L power:GND #PWR2
 U 1 1 57C960BE
 P 4300 3700
@@
 $EndComp
 $Comp
-L GND #PWR3
+L power:GND #PWR3
 U 1 1 57C99E1F
 P 4300 5100
@@
 $EndComp
 $Comp
-L GND #PWR7
+L power:GND #PWR7
 U 1 1 57C9A3C2
 P 4800 6100
@@
 $EndComp
 $Comp
-L GND #PWR6
+L power:GND #PWR6
 U 1 1 57CA25EF
 P 4800 3900
@@
 MT-IN-R-2
 $Comp
-L C_Small C3
+L KERISEv1-rescue:C_Small C3
 U 1 1 57CCF51A
 P 4500 1500
@@
 $EndComp
 $Comp
-L C_Small C4
+L KERISEv1-rescue:C_Small C4
 U 1 1 57CDA654
 P 4500 1700
@@
 $EndComp
 $Comp
-L C_Small C2
+L KERISEv1-rescue:C_Small C2
 U 1 1 57CDA6E0
 P 4500 1300
@@
 $EndComp
 $Comp
-L C_Small C1
+L KERISEv1-rescue:C_Small C1
 U 1 1 57CDA771
 P 4500 1100
@@
 $EndComp
 $Comp
-L C_Small C5
+L KERISEv1-rescue:C_Small C5
 U 1 1 57CDA805
 P 4500 2000
@@
 $EndComp
 $Comp
-L GND #PWR1
+L power:GND #PWR1
 U 1 1 57CDA895
 P 4300 2600
@@
 $EndComp
 $Comp
-L C_Small C6
+L KERISEv1-rescue:C_Small C6
 U 1 1 57CDB4B2
 P 4500 2300
@@
 RESET
 $Comp
-L C C9
+L KERISEv1-rescue:C C9
 U 1 1 57CDEB3C
 P 4600 3300
@@
 SPEAKER
 $Comp
-L PWR_FLAG #FLG1
+L power:PWR_FLAG #FLG1
 U 1 1 57D09A39
 P 4700 4450
@@
 $EndComp
 $Comp
-L PWR_FLAG #FLG2
+L power:PWR_FLAG #FLG2
 U 1 1 57D180C1
 P 4700 4900
@@
 NoConn ~ 10300 6200
 Wire Wire Line
-	4800 1000 4800 2300
-Wire Wire Line
-	4600 1500 4900 1500
+	4800 1000 4800 1100
+Wire Wire Line
+	4600 1500 4800 1500
 Connection ~ 4800 1500
 Wire Wire Line
-	4600 1700 4900 1700
+	4600 1700 4800 1700
 Connection ~ 4800 1700
 Wire Wire Line
-	4600 2000 4900 2000
-Wire Wire Line
-	4600 2300 4900 2300
+	4600 2000 4800 2000
+Wire Wire Line
+	4600 2300 4800 2300
 Connection ~ 4800 2000
 Wire Wire Line
-	4800 5500 4800 6100
+	4800 5500 4800 5700
 Wire Wire Line
 	4800 5700 4900 5700
@@
 	3000 5300 3100 5300
 Wire Wire Line
-	4600 1100 4900 1100
-Wire Wire Line
-	4600 1300 4900 1300
+	4600 1100 4800 1100
+Wire Wire Line
+	4600 1300 4800 1300
 Connection ~ 4800 1100
 Connection ~ 4800 1300
@@
 Connection ~ 4800 6000
 Wire Wire Line
-	4300 1100 4300 2600
+	4300 1100 4300 1300
 Wire Wire Line
 	4300 2000 4400 2000
@@
 	2300 2200 2400 2200
 Wire Wire Line
-	4200 2900 4900 2900
+	4200 2900 4300 2900
 Wire Wire Line
 	4300 3700 4300 3600
@@
 	4700 4450 4700 4550
 Wire Wire Line
-	4600 4550 4900 4550
-Wire Wire Line
-	4300 4550 4300 5100
+	4600 4550 4700 4550
+Wire Wire Line
+	4300 4550 4300 4800
 Wire Wire Line
 	4300 4800 4400 4800
@@
 Connection ~ 4700 4550
 Wire Wire Line
-	4600 4800 4900 4800
+	4600 4800 4700 4800
 Wire Wire Line
 	4700 4800 4700 4900
@@
 	10300 800  10400 800
 $Comp
-L Tactile_SW_4P SW1
+L KERISEv1:Tactile_SW_4P SW1
 U 1 1 57DDDB01
 P 3900 3300
@@
 Main
 $Comp
-L STM32F405RGTx-RESCUE-KERISEv1 U1
+L KERISEv1-rescue:STM32F405RGTx-RESCUE-KERISEv1 U1
 U 1 1 5862791B
 P 7600 3600
@@
 	1    0    0    -1
 $EndComp
+Wire Wire Line
+	4800 1500 4800 1700
+Wire Wire Line
+	4800 1500 4900 1500
+Wire Wire Line
+	4800 1700 4900 1700
+Wire Wire Line
+	4800 1700 4800 2000
+Wire Wire Line
+	4800 2000 4900 2000
+Wire Wire Line
+	4800 2000 4800 2300
+Wire Wire Line
+	4800 5700 4800 6000
+Wire Wire Line
+	4800 1100 4800 1300
+Wire Wire Line
+	4800 1100 4900 1100
+Wire Wire Line
+	4800 1300 4900 1300
+Wire Wire Line
+	4800 1300 4800 1500
+Wire Wire Line
+	4800 6000 4800 6100
+Wire Wire Line
+	4300 2000 4300 2300
+Wire Wire Line
+	4300 1700 4300 2000
+Wire Wire Line
+	4300 1500 4300 1700
+Wire Wire Line
+	4300 1300 4300 1500
+Wire Wire Line
+	4800 2300 4900 2300
+Wire Wire Line
+	4300 2300 4300 2600
+Wire Wire Line
+	4600 2900 4900 2900
+Wire Wire Line
+	4300 2900 4600 2900
+Wire Wire Line
+	4300 4800 4300 5100
+Wire Wire Line
+	4700 4550 4900 4550
+Wire Wire Line
+	4700 4800 4900 4800
 $EndSCHEMATC
