File: kicad/Power.sch (KiCad schematic (older format))
At the start: 20 parts, among them P3 Battery_A, P4 Battery_B, SW2 Power, U4 LXDC55FAAA-203, U5 REF1933, U6 LT1963ES8

Commit message: KiCadデータの名前をKERISEv1に変更
Parts:
- removed U4: LXDC55FAAA-203, kerikun11:LXDC55FAAA-203, symbol LXDC55FAAA-203
- added U?: LXDC55FAAA-203, symbol LXDC55FAAA-203
Changed lines of the file:
@@
 EESchema Schematic File Version 2
-LIBS:Mouse-01
 LIBS:74xgxx
 LIBS:74xx
@@
 LIBS:xilinx
 LIBS:Zilog
-LIBS:Mouse-01-cache
+LIBS:KERISEv1
+LIBS:kerikun11
+LIBS:KERISEv1-cache
 EELAYER 25 0
 EELAYER END
@@
 Comment4 ""
 $EndDescr
-$Comp
-L LXDC55FAAA-203 U4
-U 1 1 57CA160F
-P 6850 3000
-F 0 "U4" H 6850 3450 60  0000 C CNN
-F 1 "LXDC55FAAA-203" H 6850 3350 60  0000 C CNN
-F 2 "kerikun11:LXDC55FAAA-203" H 6850 3300 60  0001 C CNN
-F 3 "" H 6850 3300 60  0000 C CNN
-	1    6850 3000
-	1    0    0    -1
-$EndComp
 Wire Wire Line
 	6100 2800 6100 3100
@@
 Connection ~ 5900 2800
 $Comp
-L GND #PWR028
+L GND #PWR33
 U 1 1 57CA1878
 P 5900 3700
-F 0 "#PWR028" H 5900 3450 50  0001 C CNN
+F 0 "#PWR33" H 5900 3450 50  0001 C CNN
 F 1 "GND" H 5900 3550 50  0000 C CNN
 F 2 "" H 5900 3700 50  0000 C CNN
@@
 	5900 3700 5900 3500
 $Comp
-L GND #PWR029
+L GND #PWR34
 U 1 1 57CA18AE
 P 6700 3700
-F 0 "#PWR029" H 6700 3450 50  0001 C CNN
+F 0 "#PWR34" H 6700 3450 50  0001 C CNN
 F 1 "GND" H 6700 3550 50  0000 C CNN
 F 2 "" H 6700 3700 50  0000 C CNN
@@
 $EndComp
 $Comp
-L GND #PWR030
+L GND #PWR35
 U 1 1 57CA1AC2
 P 8000 3700
-F 0 "#PWR030" H 8000 3450 50  0001 C CNN
+F 0 "#PWR35" H 8000 3450 50  0001 C CNN
 F 1 "GND" H 8000 3550 50  0000 C CNN
 F 2 "" H 8000 3700 50  0000 C CNN
@@
 Connection ~ 7600 2900
 $Comp
-L +5V #PWR031
+L +5V #PWR29
 U 1 1 57CA2050
 P 8600 2700
-F 0 "#PWR031" H 8600 2550 50  0001 C CNN
+F 0 "#PWR29" H 8600 2550 50  0001 C CNN
 F 1 "+5V" H 8600 2840 50  0000 C CNN
 F 2 "" H 8600 2700 50  0000 C CNN
@@
 	8600 2700 8600 3200
 $Comp
-L +BATT #PWR032
+L +BATT #PWR28
 U 1 1 57CA210F
 P 5900 2700
-F 0 "#PWR032" H 5900 2550 50  0001 C CNN
+F 0 "#PWR28" H 5900 2550 50  0001 C CNN
 F 1 "+BATT" H 5900 2840 50  0000 C CNN
 F 2 "" H 5900 2700 50  0000 C CNN
@@
 $EndComp
 $Comp
-L GND #PWR033
+L GND #PWR36
 U 1 1 57CA23AF
 P 8300 3700
-F 0 "#PWR033" H 8300 3450 50  0001 C CNN
+F 0 "#PWR36" H 8300 3450 50  0001 C CNN
 F 1 "GND" H 8300 3550 50  0000 C CNN
 F 2 "" H 8300 3700 50  0000 C CNN
@@
 $EndComp
 $Comp
-L GND #PWR034
+L GND #PWR37
 U 1 1 57CA271B
 P 8600 3700
-F 0 "#PWR034" H 8600 3450 50  0001 C CNN
+F 0 "#PWR37" H 8600 3450 50  0001 C CNN
 F 1 "GND" H 8600 3550 50  0000 C CNN
 F 2 "" H 8600 3700 50  0000 C CNN
@@
 	8000 3200 8000 3300
 $Comp
-L +BATT #PWR035
+L +BATT #PWR26
 U 1 1 57CC111A
 P 4900 2700
-F 0 "#PWR035" H 4900 2550 50  0001 C CNN
+F 0 "#PWR26" H 4900 2550 50  0001 C CNN
 F 1 "+BATT" H 4900 2840 50  0000 C CNN
 F 2 "" H 4900 2700 50  0000 C CNN
@@
 $EndComp
 $Comp
-L GND #PWR036
+L GND #PWR31
 U 1 1 57CC113A
 P 3800 3700
-F 0 "#PWR036" H 3800 3450 50  0001 C CNN
+F 0 "#PWR31" H 3800 3450 50  0001 C CNN
 F 1 "GND" H 3800 3550 50  0000 C CNN
 F 2 "" H 3800 3700 50  0000 C CNN
@@
 	3800 2900 3700 2900
 $Comp
-L +5V #PWR037
+L +5V #PWR40
 U 1 1 57CC1940
 P 4100 4400
-F 0 "#PWR037" H 4100 4250 50  0001 C CNN
+F 0 "#PWR40" H 4100 4250 50  0001 C CNN
 F 1 "+5V" H 4100 4540 50  0000 C CNN
 F 2 "" H 4100 4400 50  0000 C CNN
@@
 Connection ~ 4100 4500
 $Comp
-L GND #PWR038
+L GND #PWR47
 U 1 1 57CC1AB4
 P 4900 5300
-F 0 "#PWR038" H 4900 5050 50  0001 C CNN
+F 0 "#PWR47" H 4900 5050 50  0001 C CNN
 F 1 "GND" H 4900 5150 50  0000 C CNN
 F 2 "" H 4900 5300 50  0000 C CNN
@@
 	4900 5300 4900 5100
 $Comp
-L GND #PWR039
+L GND #PWR46
 U 1 1 57CC1B19
 P 4100 5300
-F 0 "#PWR039" H 4100 5050 50  0001 C CNN
+F 0 "#PWR46" H 4100 5050 50  0001 C CNN
 F 1 "GND" H 4100 5150 50  0000 C CNN
 F 2 "" H 4100 5300 50  0000 C CNN
@@
 	4100 5300 4100 5100
 $Comp
-L +3.3VA #PWR040
+L +3.3VA #PWR41
 U 1 1 57CC1D9F
 P 5600 4400
-F 0 "#PWR040" H 5750 4350 50  0001 C CNN
+F 0 "#PWR41" H 5750 4350 50  0001 C CNN
 F 1 "+3.3VA" H 5600 4500 50  0000 C CNN
 F 2 "" H 5600 4400 50  0000 C CNN
@@
 	5600 4500 5400 4500
 $Comp
-L +1.65VA #PWR041
+L +1.65VA #PWR42
 U 1 1 57CC1DFF
 P 6000 4400
-F 0 "#PWR041" H 6150 4350 50  0001 C CNN
+F 0 "#PWR42" H 6150 4350 50  0001 C CNN
 F 1 "+1.65VA" H 6000 4500 50  0000 C CNN
 F 2 "" H 6000 4400 50  0000 C CNN
@@
 $EndComp
 $Comp
-L +5V #PWR042
+L +5V #PWR43
 U 1 1 57CC204D
 P 6600 4400
-F 0 "#PWR042" H 6600 4250 50  0001 C CNN
+F 0 "#PWR43" H 6600 4250 50  0001 C CNN
 F 1 "+5V" H 6600 4540 50  0000 C CNN
 F 2 "" H 6600 4400 50  0000 C CNN
@@
 $EndComp
 $Comp
-L GND #PWR043
+L GND #PWR50
 U 1 1 57CC212C
 P 6600 5300
-F 0 "#PWR043" H 6600 5050 50  0001 C CNN
+F 0 "#PWR50" H 6600 5050 50  0001 C CNN
 F 1 "GND" H 6600 5150 50  0000 C CNN
 F 2 "" H 6600 5300 50  0000 C CNN
@@
 Connection ~ 6900 4500
 $Comp
-L GND #PWR044
+L GND #PWR51
 U 1 1 57CC2261
 P 7600 5300
-F 0 "#PWR044" H 7600 5050 50  0001 C CNN
+F 0 "#PWR51" H 7600 5050 50  0001 C CNN
 F 1 "GND" H 7600 5150 50  0000 C CNN
 F 2 "" H 7600 5300 50  0000 C CNN
@@
 	7700 5200 7700 5100
 $Comp
-L +3.3V #PWR045
+L +3.3V #PWR44
 U 1 1 57CC235F
 P 8500 4400
-F 0 "#PWR045" H 8500 4250 50  0001 C CNN
+F 0 "#PWR44" H 8500 4250 50  0001 C CNN
 F 1 "+3.3V" H 8500 4540 50  0000 C CNN
 F 2 "" H 8500 4400 50  0000 C CNN
@@
 $EndComp
 $Comp
-L GND #PWR046
+L GND #PWR52
 U 1 1 57CC26B1
 P 8500 5300
-F 0 "#PWR046" H 8500 5050 50  0001 C CNN
+F 0 "#PWR52" H 8500 5050 50  0001 C CNN
 F 1 "GND" H 8500 5150 50  0000 C CNN
 F 2 "" H 8500 5300 50  0000 C CNN
@@
 Connection ~ 6000 4600
 $Comp
-L GND #PWR047
+L GND #PWR48
 U 1 1 57CC28D4
 P 5600 5300
-F 0 "#PWR047" H 5600 5050 50  0001 C CNN
+F 0 "#PWR48" H 5600 5050 50  0001 C CNN
 F 1 "GND" H 5600 5150 50  0000 C CNN
 F 2 "" H 5600 5300 50  0000 C CNN
@@
 	5600 5300 5600 5100
 $Comp
-L GND #PWR048
+L GND #PWR49
 U 1 1 57CC2961
 P 6000 5300
-F 0 "#PWR048" H 6000 5050 50  0001 C CNN
+F 0 "#PWR49" H 6000 5050 50  0001 C CNN
 F 1 "GND" H 6000 5150 50  0000 C CNN
 F 2 "" H 6000 5300 50  0000 C CNN
@@
 $EndComp
 $Comp
-L GND #PWR049
+L GND #PWR32
 U 1 1 57CD3C05
 P 5200 3700
-F 0 "#PWR049" H 5200 3450 50  0001 C CNN
+F 0 "#PWR32" H 5200 3450 50  0001 C CNN
 F 1 "GND" H 5200 3550 50  0000 C CNN
 F 2 "" H 5200 3700 50  0000 C CNN
@@
 	5200 3600 5200 3700
 $Comp
-L +BATT #PWR050
+L +BATT #PWR27
 U 1 1 57CD3CA2
 P 5200 2700
-F 0 "#PWR050" H 5200 2550 50  0001 C CNN
+F 0 "#PWR27" H 5200 2550 50  0001 C CNN
 F 1 "+BATT" H 5200 2840 50  0000 C CNN
 F 2 "" H 5200 2700 50  0000 C CNN
@@
 NoConn ~ 4800 2800
 $Comp
-L GND #PWR051
+L GND #PWR45
 U 1 1 57D18DB8
 P 3600 5300
-F 0 "#PWR051" H 3600 5050 50  0001 C CNN
+F 0 "#PWR45" H 3600 5050 50  0001 C CNN
 F 1 "GND" H 3600 5150 50  0000 C CNN
 F 2 "" H 3600 5300 50  0000 C CNN
@@
 $EndComp
 $Comp
-L PWR_FLAG #FLG052
+L PWR_FLAG #FLG4
 U 1 1 57D18DE7
 P 3600 5200
-F 0 "#FLG052" H 3600 5295 50  0001 C CNN
+F 0 "#FLG4" H 3600 5295 50  0001 C CNN
 F 1 "PWR_FLAG" H 3600 5380 50  0000 C CNN
 F 2 "" H 3600 5200 50  0000 C CNN
@@
 	3600 5200 3600 5300
 $Comp
-L PWR_FLAG #FLG053
+L PWR_FLAG #FLG3
 U 1 1 57D1915C
 P 3600 4500
-F 0 "#FLG053" H 3600 4595 50  0001 C CNN
+F 0 "#FLG3" H 3600 4595 50  0001 C CNN
 F 1 "PWR_FLAG" H 3600 4680 50  0000 C CNN
 F 2 "" H 3600 4500 50  0000 C CNN
@@
 $EndComp
 $Comp
-L +BATT #PWR054
+L +BATT #PWR39
 U 1 1 57D1923B
 P 3600 4400
-F 0 "#PWR054" H 3600 4250 50  0001 C CNN
+F 0 "#PWR39" H 3600 4250 50  0001 C CNN
 F 1 "+BATT" H 3600 4540 50  0000 C CNN
 F 2 "" H 3600 4400 50  0000 C CNN
@@
 $EndComp
 $Comp
-L +5V #PWR055
+L +5V #PWR30
 U 1 1 57D009FE
 P 9100 2700
-F 0 "#PWR055" H 9100 2550 50  0001 C CNN
+F 0 "#PWR30" H 9100 2550 50  0001 C CNN
 F 1 "+5V" H 9100 2840 50  0000 C CNN
 F 2 "" H 9100 2700 50  0000 C CNN
@@
 $EndComp
 $Comp
-L GND #PWR056
+L GND #PWR38
 U 1 1 57D00A42
 P 9100 3700
-F 0 "#PWR056" H 9100 3450 50  0001 C CNN
+F 0 "#PWR38" H 9100 3450 50  0001 C CNN
 F 1 "GND" H 9100 3550 50  0000 C CNN
 F 2 "" H 9100 3700 50  0000 C CNN
@@
 Wire Wire Line
 	3800 3400 3700 3400
+$Comp
+L LXDC55FAAA-203 U?
+U 1 1 58627F28
+P 6850 3000
+F 0 "U?" H 6850 3450 60  0000 C CNN
+F 1 "LXDC55FAAA-203" H 6850 3350 60  0000 C CNN
+F 2 "" H 6850 3300 60  0000 C CNN
+F 3 "" H 6850 3300 60  0000 C CNN
+	1    6850 3000
+	1    0    0    -1
+$EndComp
 $EndSCHEMATC

Commit message: 回路図を修正
電源スイッチにPchFETを挿入
赤外線LED用FETのゲートをプルダウン
Parts:
- removed SW2: Power, Pin_Headers:Pin_Header_Straight_1x03, symbol SWITCH_INV
- added C13: 0.1u, symbol C
- added Q1: IRLML6402, symbol Q_PMOS_DGS
- added R1: 10k, symbol R
- added SW2: SW_SPDT, symbol SW_SPDT
- D1: symbol LED -> LED-RESCUE-KERISEv1
- gave numbers to parts that had none: 1
- renumbered C15 to C12, C16 to C14, C12 to C15, C17 to C16, C18 to C17, C13 to C18, C14 to C19, C19 to C20, R1 to R3, R3 to R5, R5 to R6, U5 to U4
Connections:
- wire segments 67 -> 73
Other:
- note added: "Power\nKERI's Lab 2017.11.3"
- note removed: "Power"
- moved on the sheet: C12, C14, C15, C16, C17, C18, C19, C20, R2, R5, R6, U4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

Commit message: add kicad .gitignore
Parts:
- C12, C13, C14, C15, C16, C17, C18, C20: symbol C -> KERISEv1-rescue:C
- C19: symbol CP -> KERISEv1-rescue:CP
- D1: symbol LED-RESCUE-KERISEv1 -> KERISEv1-rescue:LED-RESCUE-KERISEv1
- P3, P4: symbol CONN_01X02 -> KERISEv1-rescue:CONN_01X02
- Q1: symbol Q_PMOS_DGS -> KERISEv1-rescue:Q_PMOS_DGS
- R1, R2, R3, R4, R5, R6: symbol R -> KERISEv1-rescue:R
- SW2: symbol SW_SPDT -> KERISEv1-rescue:SW_SPDT
- U4: symbol REF1933 -> KERISEv1:REF1933
- U5: symbol LXDC55FAAA-203 -> KERISEv1-rescue:LXDC55FAAA-203
- U6: symbol LT1963ES8 -> KERISEv1:LT1963ES8
