File: kicad/UI.sch (KiCad schematic (older format))
At the start: 14 parts, among them Q3 BSS138, SW3 BUTTON

Commit message: 回路図を修正
電源スイッチにPchFETを挿入
赤外線LED用FETのゲートをプルダウン
Parts:
- D10, D11, D12, D13: symbol LED -> LED-RESCUE-KERISEv1
- renumbered C31 to C32, Q3 to Q4, R23 to R21, R19 to R22, R20 to R23, R21 to R24, R22 to R25, R18 to R26
Changed lines of the file:
@@
 EESchema Schematic File Version 2
+LIBS:KERISEv1-rescue
 LIBS:74xgxx
 LIBS:74xx
@@
 LIBS:cmos4000
 LIBS:conn
-LIBS:connectors
 LIBS:contrib
 LIBS:cypress
@@
 LIBS:ftdi
 LIBS:gennum
-LIBS:graphic
 LIBS:hc11
-LIBS:ic-cpu
-LIBS:ic-io
-LIBS:ic-misc
-LIBS:ic-power
 LIBS:intel
 LIBS:interface
@@
 LIBS:Lattice
 LIBS:linear
-LIBS:logo
 LIBS:maxim
 LIBS:memory
@@
 LIBS:opto
 LIBS:Oscillators
-LIBS:passive
 LIBS:philips
 LIBS:power
@@
 LIBS:Zilog
 LIBS:KERISEv1
-LIBS:kerikun11
 LIBS:KERISEv1-cache
 EELAYER 25 0
@@
 $EndComp
 $Comp
-L +3.3V #PWR85
+L +3.3V #PWR89
 U 1 1 57CE7538
 P 4400 3500
-F 0 "#PWR85" H 4400 3350 50  0001 C CNN
+F 0 "#PWR89" H 4400 3350 50  0001 C CNN
 F 1 "+3.3V" H 4400 3640 50  0000 C CNN
 F 2 "" H 4400 3500 50  0000 C CNN
@@
 $EndComp
 $Comp
-L R R23
+L R R21
 U 1 1 57CE757A
 P 4000 4450
-F 0 "R23" V 4080 4450 50  0000 C CNN
+F 0 "R21" V 4080 4450 50  0000 C CNN
 F 1 "4.7k" V 4000 4450 50  0000 C CNN
 F 2 "Resistors_SMD:R_0603" V 3930 4450 50  0001 C CNN
@@
 $EndComp
 $Comp
-L Q_NMOS_GSD Q3
+L Q_NMOS_GSD Q4
 U 1 1 57CE75AD
 P 4300 4200
-F 0 "Q3" H 4600 4250 50  0000 R CNN
+F 0 "Q4" H 4600 4250 50  0000 R CNN
 F 1 "BSS138" H 4800 4150 50  0000 R CNN
 F 2 "TO_SOT_Packages_SMD:SOT-23" H 4500 4300 50  0001 C CNN
@@
 $EndComp
 $Comp
-L GND #PWR87
+L GND #PWR90
 U 1 1 57CE7673
 P 4400 4700
-F 0 "#PWR87" H 4400 4450 50  0001 C CNN
+F 0 "#PWR90" H 4400 4450 50  0001 C CNN
 F 1 "GND" H 4400 4550 50  0000 C CNN
 F 2 "" H 4400 4700 50  0000 C CNN
@@
 $EndComp
 $Comp
-L GND #PWR86
+L GND #PWR88
 U 1 1 57CE768B
 P 4000 4700
-F 0 "#PWR86" H 4000 4450 50  0001 C CNN
+F 0 "#PWR88" H 4000 4450 50  0001 C CNN
 F 1 "GND" H 4000 4550 50  0000 C CNN
 F 2 "" H 4000 4700 50  0000 C CNN
@@
 Connection ~ 4000 4200
 $Comp
-L LED D10
+L LED-RESCUE-KERISEv1 D10
 U 1 1 57CE80D9
 P 6000 4400
@@
 $EndComp
 $Comp
-L LED D11
+L LED-RESCUE-KERISEv1 D11
 U 1 1 57CE812A
 P 6300 4400
@@
 $EndComp
 $Comp
-L LED D12
+L LED-RESCUE-KERISEv1 D12
 U 1 1 57CE815D
 P 6600 4400
@@
 $EndComp
 $Comp
-L LED D13
+L LED-RESCUE-KERISEv1 D13
 U 1 1 57CE8187
 P 6900 4400
@@
 $EndComp
 $Comp
-L GND #PWR88
+L GND #PWR91
 U 1 1 57CE8530
 P 6000 4700
-F 0 "#PWR88" H 6000 4450 50  0001 C CNN
+F 0 "#PWR91" H 6000 4450 50  0001 C CNN
 F 1 "GND" H 6000 4550 50  0000 C CNN
 F 2 "" H 6000 4700 50  0000 C CNN
@@
 $EndComp
 $Comp
-L GND #PWR89
+L GND #PWR92
 U 1 1 57CE8557
 P 6300 4700
-F 0 "#PWR89" H 6300 4450 50  0001 C CNN
+F 0 "#PWR92" H 6300 4450 50  0001 C CNN
 F 1 "GND" H 6300 4550 50  0000 C CNN
 F 2 "" H 6300 4700 50  0000 C CNN
@@
 $EndComp
 $Comp
-L GND #PWR90
+L GND #PWR93
 U 1 1 57CE8577
 P 6600 4700
-F 0 "#PWR90" H 6600 4450 50  0001 C CNN
+F 0 "#PWR93" H 6600 4450 50  0001 C CNN
 F 1 "GND" H 6600 4550 50  0000 C CNN
 F 2 "" H 6600 4700 50  0000 C CNN
@@
 $EndComp
 $Comp
-L GND #PWR91
+L GND #PWR94
 U 1 1 57CE8597
 P 6900 4700
-F 0 "#PWR91" H 6900 4450 50  0001 C CNN
+F 0 "#PWR94" H 6900 4450 50  0001 C CNN
 F 1 "GND" H 6900 4550 50  0000 C CNN
 F 2 "" H 6900 4700 50  0000 C CNN
@@
 	6000 4600 6000 4700
 $Comp
-L R R19
+L R R22
 U 1 1 57CE8600
 P 6000 3950
-F 0 "R19" V 6080 3950 50  0000 C CNN
+F 0 "R22" V 6080 3950 50  0000 C CNN
 F 1 "1k" V 6000 3950 50  0000 C CNN
 F 2 "Resistors_SMD:R_0603" V 5930 3950 50  0001 C CNN
@@
 $EndComp
 $Comp
-L R R20
+L R R23
 U 1 1 57CE8644
 P 6300 3950
-F 0 "R20" V 6380 3950 50  0000 C CNN
+F 0 "R23" V 6380 3950 50  0000 C CNN
 F 1 "1k" V 6300 3950 50  0000 C CNN
 F 2 "Resistors_SMD:R_0603" V 6230 3950 50  0001 C CNN
@@
 $EndComp
 $Comp
-L R R21
+L R R24
 U 1 1 57CE8677
 P 6600 3950
-F 0 "R21" V 6680 3950 50  0000 C CNN
+F 0 "R24" V 6680 3950 50  0000 C CNN
 F 1 "1k" V 6600 3950 50  0000 C CNN
 F 2 "Resistors_SMD:R_0603" V 6530 3950 50  0001 C CNN
@@
 $EndComp
 $Comp
-L R R22
+L R R25
 U 1 1 57CE86AD
 P 6900 3950
-F 0 "R22" V 6980 3950 50  0000 C CNN
+F 0 "R25" V 6980 3950 50  0000 C CNN
 F 1 "1k" V 6900 3950 50  0000 C CNN
 F 2 "Resistors_SMD:R_0603" V 6830 3950 50  0001 C CNN
@@
 	6900 3400 6900 3800
 $Comp
-L GND #PWR92
+L GND #PWR96
 U 1 1 57CEA2EF
 P 8200 4700
-F 0 "#PWR92" H 8200 4450 50  0001 C CNN
+F 0 "#PWR96" H 8200 4450 50  0001 C CNN
 F 1 "GND" H 8200 4550 50  0000 C CNN
 F 2 "" H 8200 4700 50  0000 C CNN
@@
 	8200 3700 8200 4000
 $Comp
-L R R18
+L R R26
 U 1 1 57CEA520
 P 8200 3550
-F 0 "R18" V 8280 3550 50  0000 C CNN
+F 0 "R26" V 8280 3550 50  0000 C CNN
 F 1 "10k" V 8200 3550 50  0000 C CNN
 F 2 "Resistors_SMD:R_0603" V 8130 3550 50  0001 C CNN
@@
 $EndComp
 $Comp
-L +3.3V #PWR84
+L +3.3V #PWR95
 U 1 1 57CEA571
 P 8200 3300
-F 0 "#PWR84" H 8200 3150 50  0001 C CNN
+F 0 "#PWR95" H 8200 3150 50  0001 C CNN
 F 1 "+3.3V" H 8200 3440 50  0000 C CNN
 F 2 "" H 8200 3300 50  0000 C CNN
@@
 Connection ~ 8200 3800
 $Comp
-L C C31
+L C C32
 U 1 1 57CEAAA3
 P 8500 4200
-F 0 "C31" H 8525 4300 50  0000 L CNN
+F 0 "C32" H 8525 4300 50  0000 L CNN
 F 1 "0.1u" H 8525 4100 50  0000 L CNN
 F 2 "Capacitors_SMD:C_0603" H 8538 4050 50  0001 C CNN
@@
 $EndComp
 $Comp
-L GND #PWR93
+L GND #PWR97
 U 1 1 57CEAAF6
 P 8500 4700
-F 0 "#PWR93" H 8500 4450 50  0001 C CNN
+F 0 "#PWR97" H 8500 4450 50  0001 C CNN
 F 1 "GND" H 8500 4550 50  0000 C CNN
 F 2 "" H 8500 4700 50  0000 C CNN

Commit message: add kicad .gitignore
Parts:
- C32: symbol C -> KERISEv1-rescue:C
- D10, D11, D12, D13: symbol LED-RESCUE-KERISEv1 -> KERISEv1-rescue:LED-RESCUE-KERISEv1
- Q4: symbol Q_NMOS_GSD -> KERISEv1-rescue:Q_NMOS_GSD
- R21, R22, R23, R24, R25, R26: symbol R -> KERISEv1-rescue:R
- SP1: symbol SPEAKER -> KERISEv1-rescue:SPEAKER
- SW3: symbol Tactile_SW_4P -> KERISEv1:Tactile_SW_4P
Changed lines of the file:
@@
-EESchema Schematic File Version 2
-LIBS:KERISEv1-rescue
-LIBS:74xgxx
-LIBS:74xx
-LIBS:ac-dc
-LIBS:actel
-LIBS:adc-dac
-LIBS:Altera
-LIBS:analog_devices
-LIBS:analog_switches
-LIBS:atmel
-LIBS:audio
-LIBS:brooktre
-LIBS:cmos_ieee
-LIBS:cmos4000
-LIBS:conn
-LIBS:contrib
-LIBS:cypress
-LIBS:dc-dc
-LIBS:device
-LIBS:digital-audio
-LIBS:diode
-LIBS:display
-LIBS:dsp
-LIBS:elec-unifil
-LIBS:ESD_Protection
-LIBS:ftdi
-LIBS:gennum
-LIBS:hc11
-LIBS:intel
-LIBS:interface
-LIBS:ir
-LIBS:Lattice
-LIBS:linear
-LIBS:maxim
-LIBS:memory
-LIBS:microchip
-LIBS:microchip_dspic33dsc
-LIBS:microchip_pic10mcu
-LIBS:microchip_pic12mcu
-LIBS:microchip_pic16mcu
-LIBS:microchip_pic18mcu
-LIBS:microchip_pic32mcu
-LIBS:microcontrollers
-LIBS:motor_drivers
-LIBS:motorola
-LIBS:msp430
-LIBS:nordicsemi
-LIBS:nxp_armmcu
-LIBS:onsemi
-LIBS:opto
-LIBS:Oscillators
-LIBS:philips
-LIBS:power
-LIBS:Power_Management
-LIBS:powerint
-LIBS:pspice
-LIBS:references
-LIBS:regul
-LIBS:relays
-LIBS:rfcom
-LIBS:sensors
-LIBS:silabs
-LIBS:siliconi
-LIBS:stm8
-LIBS:stm32
-LIBS:supertex
-LIBS:switches
-LIBS:texas
-LIBS:transf
-LIBS:transistors
-LIBS:ttl_ieee
-LIBS:valves
-LIBS:video
-LIBS:Xicor
-LIBS:xilinx
-LIBS:Zilog
-LIBS:KERISEv1
-LIBS:KERISEv1-cache
-EELAYER 25 0
+EESchema Schematic File Version 4
+EELAYER 30 0
 EELAYER END
 $Descr A4 11693 8268
@@
 $EndDescr
 $Comp
-L SPEAKER SP1
+L KERISEv1-rescue:SPEAKER SP1
 U 1 1 57CD8DE7
 P 4800 3700
+AR Path="/57CD8DE7" Ref="SP1"  Part="1"
+AR Path="/57CD8D81/57CD8DE7" Ref="SP1"  Part="1"
 F 0 "SP1" H 4700 3950 50  0000 C CNN
 F 1 "SMT-0440" H 4700 3450 50  0000 C CNN
@@
 $EndComp
 $Comp
-L +3.3V #PWR89
+L power:+3.3V #PWR89
 U 1 1 57CE7538
 P 4400 3500
@@
 $EndComp
 $Comp
-L R R21
+L KERISEv1-rescue:R R21
 U 1 1 57CE757A
 P 4000 4450
+AR Path="/57CE757A" Ref="R21"  Part="1"
+AR Path="/57CD8D81/57CE757A" Ref="R21"  Part="1"
 F 0 "R21" V 4080 4450 50  0000 C CNN
 F 1 "4.7k" V 4000 4450 50  0000 C CNN
@@
 $EndComp
 $Comp
-L Q_NMOS_GSD Q4
+L KERISEv1-rescue:Q_NMOS_GSD Q4
 U 1 1 57CE75AD
 P 4300 4200
+AR Path="/57CE75AD" Ref="Q4"  Part="1"
+AR Path="/57CD8D81/57CE75AD" Ref="Q4"  Part="1"
 F 0 "Q4" H 4600 4250 50  0000 R CNN
 F 1 "BSS138" H 4800 4150 50  0000 R CNN
@@
 $EndComp
 $Comp
-L GND #PWR90
+L power:GND #PWR90
 U 1 1 57CE7673
 P 4400 4700
@@
 $EndComp
 $Comp
-L GND #PWR88
+L power:GND #PWR88
 U 1 1 57CE768B
 P 4000 4700
@@
 	4400 4400 4400 4700
 Wire Wire Line
-	3900 4200 4100 4200
+	3900 4200 4000 4200
 Wire Wire Line
 	4000 4200 4000 4300
@@
 Connection ~ 4000 4200
 $Comp
-L LED-RESCUE-KERISEv1 D10
+L KERISEv1-rescue:LED-RESCUE-KERISEv1 D10
 U 1 1 57CE80D9
 P 6000 4400
@@
 $EndComp
 $Comp
-L LED-RESCUE-KERISEv1 D11
+L KERISEv1-rescue:LED-RESCUE-KERISEv1 D11
 U 1 1 57CE812A
 P 6300 4400
@@
 $EndComp
 $Comp
-L LED-RESCUE-KERISEv1 D12
+L KERISEv1-rescue:LED-RESCUE-KERISEv1 D12
 U 1 1 57CE815D
 P 6600 4400
@@
 $EndComp
 $Comp
-L LED-RESCUE-KERISEv1 D13
+L KERISEv1-rescue:LED-RESCUE-KERISEv1 D13
 U 1 1 57CE8187
 P 6900 4400
@@
 $EndComp
 $Comp
-L GND #PWR91
+L power:GND #PWR91
 U 1 1 57CE8530
 P 6000 4700
@@
 $EndComp
 $Comp
-L GND #PWR92
+L power:GND #PWR92
 U 1 1 57CE8557
 P 6300 4700
@@
 $EndComp
 $Comp
-L GND #PWR93
+L power:GND #PWR93
 U 1 1 57CE8577
 P 6600 4700
@@
 $EndComp
 $Comp
-L GND #PWR94
+L power:GND #PWR94
 U 1 1 57CE8597
 P 6900 4700
@@
 	6000 4600 6000 4700
 $Comp
-L R R22
+L KERISEv1-rescue:R R22
 U 1 1 57CE8600
 P 6000 3950
+AR Path="/57CE8600" Ref="R22"  Part="1"
+AR Path="/57CD8D81/57CE8600" Ref="R22"  Part="1"
 F 0 "R22" V 6080 3950 50  0000 C CNN
 F 1 "1k" V 6000 3950 50  0000 C CNN
@@
 $EndComp
 $Comp
-L R R23
+L KERISEv1-rescue:R R23
 U 1 1 57CE8644
 P 6300 3950
+AR Path="/57CE8644" Ref="R23"  Part="1"
+AR Path="/57CD8D81/57CE8644" Ref="R23"  Part="1"
 F 0 "R23" V 6380 3950 50  0000 C CNN
 F 1 "1k" V 6300 3950 50  0000 C CNN
@@
 $EndComp
 $Comp
-L R R24
+L KERISEv1-rescue:R R24
 U 1 1 57CE8677
 P 6600 3950
+AR Path="/57CE8677" Ref="R24"  Part="1"
+AR Path="/57CD8D81/57CE8677" Ref="R24"  Part="1"
 F 0 "R24" V 6680 3950 50  0000 C CNN
 F 1 "1k" V 6600 3950 50  0000 C CNN
@@
 $EndComp
 $Comp
-L R R25
+L KERISEv1-rescue:R R25
 U 1 1 57CE86AD
 P 6900 3950
+AR Path="/57CE86AD" Ref="R25"  Part="1"
+AR Path="/57CD8D81/57CE86AD" Ref="R25"  Part="1"
 F 0 "R25" V 6980 3950 50  0000 C CNN
 F 1 "1k" V 6900 3950 50  0000 C CNN
@@
 	6900 3400 6900 3800
 $Comp
-L GND #PWR96
+L power:GND #PWR96
 U 1 1 57CEA2EF
 P 8200 4700
@@
 BUTTON
 Wire Wire Line
-	8100 3800 8500 3800
-Wire Wire Line
-	8200 3700 8200 4000
-$Comp
-L R R26
+	8100 3800 8200 3800
+Wire Wire Line
+	8200 3700 8200 3800
+$Comp
+L KERISEv1-rescue:R R26
 U 1 1 57CEA520
 P 8200 3550
+AR Path="/57CEA520" Ref="R26"  Part="1"
+AR Path="/57CD8D81/57CEA520" Ref="R26"  Part="1"
 F 0 "R26" V 8280 3550 50  0000 C CNN
 F 1 "10k" V 8200 3550 50  0000 C CNN
@@
 $EndComp
 $Comp
-L +3.3V #PWR95
+L power:+3.3V #PWR95
 U 1 1 57CEA571
 P 8200 3300
@@
 Connection ~ 8200 3800
 $Comp
-L C C32
+L KERISEv1-rescue:C C32
 U 1 1 57CEAAA3
 P 8500 4200
+AR Path="/57CEAAA3" Ref="C32"  Part="1"
+AR Path="/57CD8D81/57CEAAA3" Ref="C32"  Part="1"
 F 0 "C32" H 8525 4300 50  0000 L CNN
 F 1 "0.1u" H 8525 4100 50  0000 L CNN
@@
 $EndComp
 $Comp
-L GND #PWR97
+L power:GND #PWR97
 U 1 1 57CEAAF6
 P 8500 4700
@@
 	8500 3800 8500 4050
 $Comp
-L Tactile_SW_4P SW3
+L KERISEv1:Tactile_SW_4P SW3
 U 1 1 57DDE1FB
 P 7800 4200
@@
 Text Notes 3300 3100 0    100  ~ 0
 User Interface
+Wire Wire Line
+	4000 4200 4100 4200
+Wire Wire Line
+	8200 3800 8500 3800
+Wire Wire Line
+	8200 3800 8200 4000
 $EndSCHEMATC
